File: ti994a-peb.sch (KiCad schematic (older format))
At the start: 24 parts, among them Q1 Q_NPN_BCE, U1 74HCT138, U2 L7805, U3 74HCT244, U4 74HCT244, U5 74HCT244, U7 74HCT245

Commit message: cleanup all outdated parts
Parts:
- removed C1, C13, C3, C4, C8: 0.1uf, Capacitor_THT:C_Rect_L4.0mm_W2.5mm_P2.50mm, symbol tipi-peb-rescue:C_Small-tipi-peb-rescue
- removed C15: 10uf, Capacitor_THT:C_Rect_L4.0mm_W2.5mm_P2.50mm, symbol tipi-peb-rescue:CP1_Small-tipi-peb-rescue
- removed C17: 22uf, Capacitor_THT:C_Rect_L4.0mm_W2.5mm_P2.50mm, symbol tipi-peb-rescue:CP1_Small-tipi-peb-rescue
- removed D1: LED_ALT, LED_THT:LED_D3.0mm, symbol tipi-peb-rescue:LED_ALT-tipi-peb-rescue
- removed Q1: Q_NPN_BCE, Package_TO_SOT_THT:TO-126-3_Vertical, symbol tipi-peb-rescue:Q_NPN_BCE-tipi-peb-rescue
- removed R1, R10, R12, R2, R3, R5: 1k, Resistor_THT:R_Axial_DIN0207_L6.3mm_D2.5mm_P7.62mm_Horizontal, symbol tipi-peb-rescue:R-tipi-peb-rescue
- removed R11: 10k, Resistor_THT:R_Axial_DIN0207_L6.3mm_D2.5mm_P7.62mm_Horizontal, symbol tipi-peb-rescue:R-tipi-peb-rescue
- removed R6: 330, Resistor_THT:R_Axial_DIN0207_L6.3mm_D2.5mm_P7.62mm_Horizontal, symbol tipi-peb-rescue:R-tipi-peb-rescue
- removed U1: 74HCT138, Package_DIP:DIP-16_W7.62mm, symbol tipi-peb-rescue:74LS138-tipi-peb-rescue
- removed U2: L7805, Package_TO_SOT_THT:TO-220-3_Horizontal_TabDown, symbol Regulator_Linear:L7805
- removed U3, U4, U5: 74HCT244, Package_DIP:DIP-20_W7.62mm, symbol tipi-peb-rescue:74HC244-tipi-peb-rescue
- removed U7: 74HCT245, Package_DIP:DIP-20_W7.62mm, symbol tipi-peb-rescue:74LS245-tipi-peb-rescue
Connections:
- no-connect marks 25 -> 15
